File: RPi_GPIO.sch (KiCad schematic (older format))
At the start: 3 parts, among them J2 RPi_GPIO

Commit message: einige bauelemente erstellt
power supply für 5v erstellt
Parts:
- gave numbers to parts that had none: 2
Changed lines of the file:
@@
 LIBS:contrib
 LIBS:valves
+LIBS:regulator
 LIBS:RPi_Hat-cache
 EELAYER 25 0
@@
 P 4000 2850
 AR Path="/5A16A976" Ref="J?"  Part="1"
-AR Path="/5515D395/5A16A976" Ref="J?"  Part="1"
-F 0 "J?" H 4078 2891 50  0000 L CNN
+AR Path="/5515D395/5A16A976" Ref="J1"  Part="1"
+F 0 "J1" H 4078 2891 50  0000 L CNN
 F 1 "CONN_01X14" H 4078 2800 50  0000 L CNN
 F 2 "Pin_Headers:Pin_Header_Straight_1x14" H 4000 2850 50  0001 C CNN
@@
 P 4000 4650
 AR Path="/5A16A97D" Ref="J?"  Part="1"
-AR Path="/5515D395/5A16A97D" Ref="J?"  Part="1"
-F 0 "J?" H 4078 4691 50  0000 L CNN
+AR Path="/5515D395/5A16A97D" Ref="J3"  Part="1"
+F 0 "J3" H 4078 4691 50  0000 L CNN
 F 1 "CONN_01X14" H 4078 4600 50  0000 L CNN
 F 2 "Pin_Headers:Pin_Header_Straight_1x14" H 4000 4650 50  0001 C CNN
@@
 GPIO_0/PWM0.0
 $Comp
-L GND #PWR?
+L GND #PWR01
 U 1 1 5A16A9A2
 P 3700 5450
-F 0 "#PWR?" H 3700 5200 50  0001 C CNN
+F 0 "#PWR01" H 3700 5200 50  0001 C CNN
 F 1 "GND" H 3705 5277 50  0000 C CNN
 F 2 "" H 3700 5450 50  0001 C CNN
@@
 	3550 3550 3800 3550
 $Comp
-L +3V3 #PWR?
+L +3V3 #PWR02
 U 1 1 5A16A9C2
 P 3550 2450
-F 0 "#PWR?" H 3550 2300 50  0001 C CNN
+F 0 "#PWR02" H 3550 2300 50  0001 C CNN
 F 1 "+3V3" V 3565 2578 50  0000 L CNN
 F 2 "" H 3550 2450 50  0001 C CNN
@@
 $EndComp
 $Comp
-L +5V #PWR?
+L +5V #PWR03
 U 1 1 5A16A9C8
 P 3550 2250
-F 0 "#PWR?" H 3550 2100 50  0001 C CNN
+F 0 "#PWR03" H 3550 2100 50  0001 C CNN
 F 1 "+5V" V 3565 2423 50  0000 C CNN
 F 2 "" H 3550 2250 50  0001 C CNN
@@
 	3550 2450 3800 2450
 $Comp
-L GND #PWR?
+L GND #PWR04
 U 1 1 5A16A9D0
 P 3700 3650
-F 0 "#PWR?" H 3700 3400 50  0001 C CNN
+F 0 "#PWR04" H 3700 3400 50  0001 C CNN
 F 1 "GND" H 3705 3477 50  0000 C CNN
 F 2 "" H 3700 3650 50  0001 C CNN
