File: Power_Supply.sch (KiCad schematic (older format))
At the start: 3 parts

Commit message: einige bauelemente erstellt
power supply für 5v erstellt
Parts:
- removed U?: regler, symbol regler
- gave numbers to parts that had none: 2
Connections:
- net labels added: +5V, D24V50F5
- wire segments 2 -> 5
Changed lines of the file:
@@
 EESchema Schematic File Version 2
-LIBS:RPi_Hat-rescue
 LIBS:power
 LIBS:device
+LIBS:switches
+LIBS:relays
+LIBS:motors
 LIBS:transistors
 LIBS:conn
@@
 LIBS:contrib
 LIBS:valves
-LIBS:RPi_Hat-cache
 EELAYER 25 0
 EELAYER END
 $Descr A4 11693 8268
 encoding utf-8
-Sheet 3 4
+Sheet 1 1
 Title ""
 Date ""
@@
 $EndDescr
 $Comp
-L Conn_01x02_Male J?
+L Conn_01x02_Male J4
 U 1 1 5A0D6BC3
 P 2000 1400
-F 0 "J?" H 2000 1500 50  0000 C CNN
+F 0 "J4" H 2000 1500 50  0000 C CNN
 F 1 "Conn_01x02_Male" H 2000 1200 50  0000 C CNN
 F 2 "" H 2000 1400 50  0001 C CNN
@@
 Powersupply_12V
 $Comp
-L +12V #PWR?
+L +12V #PWR1
 U 1 1 5A0D6BCB
 P 2550 1400
-F 0 "#PWR?" H 2550 1250 50  0001 C CNN
+F 0 "#PWR1" H 2550 1250 50  0001 C CNN
 F 1 "+12V" H 2550 1540 50  0000 C CNN
 F 2 "" H 2550 1400 50  0001 C CNN
@@
 	2550 1500 2200 1500
 $Comp
-L GNDREF #PWR?
+L GNDREF #PWR3
 U 1 1 5A0D6BD3
 P 2550 1500
-F 0 "#PWR?" H 2550 1250 50  0001 C CNN
+F 0 "#PWR3" H 2550 1250 50  0001 C CNN
 F 1 "GNDREF" H 2550 1350 50  0000 C CNN
 F 2 "" H 2550 1500 50  0001 C CNN
@@
 $EndComp
 $Comp
-L Conn_01x02_Male J?
+L Conn_01x02_Male J5
 U 1 1 5A0D6BD9
 P 2000 1400
-F 0 "J?" H 2000 1500 50  0000 C CNN
+F 0 "J5" H 2000 1500 50  0000 C CNN
 F 1 "Conn_01x02_Male" H 2000 1200 50  0000 C CNN
 F 2 "" H 2000 1400 50  0001 C CNN
@@
 Powersupply_12V
 $Comp
-L +12V #PWR?
+L +12V #PWR2
 U 1 1 5A0D6BE1
 P 2550 1400
-F 0 "#PWR?" H 2550 1250 50  0001 C CNN
+F 0 "#PWR2" H 2550 1250 50  0001 C CNN
 F 1 "+12V" H 2550 1540 50  0000 C CNN
 F 2 "" H 2550 1400 50  0001 C CNN
@@
 $EndComp
 $Comp
-L GNDREF #PWR?
+L GNDREF #PWR4
 U 1 1 5A0D6BE9
 P 2550 1500
-F 0 "#PWR?" H 2550 1250 50  0001 C CNN
+F 0 "#PWR4" H 2550 1250 50  0001 C CNN
 F 1 "GNDREF" H 2550 1350 50  0000 C CNN
 F 2 "" H 2550 1500 50  0001 C CNN
@@
 $EndComp
 $Comp
-L regler U?
-U 1 1 5A0EBB70
-P 3700 1000
-F 0 "U?" H 3300 1100 60  0000 C CNN
-F 1 "regler" H 3700 1000 60  0000 C CNN
-F 2 "" H 3700 1000 60  0001 C CNN
-F 3 "" H 3700 1000 60  0001 C CNN
-	1    3700 1000
+L D24V50F5 #U09
+U 1 1 5A193EAE
+P 3900 2700
+F 0 "#U09" H 3750 2925 50  0001 C CNN
+F 1 "D24V50F5" H 3900 2925 50  0000 L CNN
+F 2 "Connectors_Samtec:SL-105-X-XX_1x05" H 3900 3025 50  0001 C CNN
+F 3 "" H 3750 2925 50  0001 C CNN
+	1    3900 2700
 	1    0    0    -1
 $EndComp
+$Comp
+L +12V #PWR5
+U 1 1 5A195F1D
+P 3400 2600
+F 0 "#PWR5" H 3400 2450 50  0001 C CNN
+F 1 "+12V" H 3400 2740 50  0000 C CNN
+F 2 "" H 3400 2600 50  0001 C CNN
+F 3 "" H 3400 2600 50  0001 C CNN
+	1    3400 2600
+	1    0    0    -1
+$EndComp
+$Comp
+L GNDREF #PWR6
+U 1 1 5A195F91
+P 3900 3100
+F 0 "#PWR6" H 3900 2850 50  0001 C CNN
+F 1 "GNDREF" H 3900 2950 50  0000 C CNN
+F 2 "" H 3900 3100 50  0001 C CNN
+F 3 "" H 3900 3100 50  0001 C CNN
+	1    3900 3100
+	1    0    0    -1
+$EndComp
+$Comp
+L +5V #PWR7
+U 1 1 5A195FAB
+P 4400 2600
+F 0 "#PWR7" H 4400 2450 50  0001 C CNN
+F 1 "+5V" H 4400 2740 50  0000 C CNN
+F 2 "" H 4400 2600 50  0001 C CNN
+F 3 "" H 4400 2600 50  0001 C CNN
+	1    4400 2600
+	1    0    0    -1
+$EndComp
+Wire Wire Line
+	4200 2600 4400 2600
+Wire Wire Line
+	3600 2600 3400 2600
+Wire Wire Line
+	3900 3000 3900 3100
 $EndSCHEMATC

Commit message: only some wires
Changed lines of the file:
@@
 EESchema Schematic File Version 2
+LIBS:RPi_Hat-rescue
 LIBS:power
 LIBS:device
-LIBS:switches
-LIBS:relays
-LIBS:motors
 LIBS:transistors
 LIBS:conn
@@
 LIBS:contrib
 LIBS:valves
+LIBS:regulator
+LIBS:RPi_Hat-cache
 EELAYER 25 0
 EELAYER END
 $Descr A4 11693 8268
 encoding utf-8
-Sheet 1 1
+Sheet 3 4
 Title ""
 Date ""
@@
 L D24V50F5 #U09
 U 1 1 5A193EAE
-P 3900 2700
-F 0 "#U09" H 3750 2925 50  0001 C CNN
-F 1 "D24V50F5" H 3900 2925 50  0000 L CNN
-F 2 "Connectors_Samtec:SL-105-X-XX_1x05" H 3900 3025 50  0001 C CNN
-F 3 "" H 3750 2925 50  0001 C CNN
-	1    3900 2700
+P 4150 1100
+F 0 "#U09" H 4000 1325 50  0001 C CNN
+F 1 "D24V50F5" H 4150 1325 50  0000 L CNN
+F 2 "Connectors_Samtec:SL-105-X-XX_1x05" H 4150 1425 50  0001 C CNN
+F 3 "" H 4000 1325 50  0001 C CNN
+	1    4150 1100
 	1    0    0    -1
 $EndComp
@@
 L +12V #PWR5
 U 1 1 5A195F1D
-P 3400 2600
-F 0 "#PWR5" H 3400 2450 50  0001 C CNN
-F 1 "+12V" H 3400 2740 50  0000 C CNN
-F 2 "" H 3400 2600 50  0001 C CNN
-F 3 "" H 3400 2600 50  0001 C CNN
-	1    3400 2600
+P 3650 1000
+F 0 "#PWR5" H 3650 850 50  0001 C CNN
+F 1 "+12V" H 3650 1140 50  0000 C CNN
+F 2 "" H 3650 1000 50  0001 C CNN
+F 3 "" H 3650 1000 50  0001 C CNN
+	1    3650 1000
 	1    0    0    -1
 $EndComp
@@
 L GNDREF #PWR6
 U 1 1 5A195F91
-P 3900 3100
-F 0 "#PWR6" H 3900 2850 50  0001 C CNN
-F 1 "GNDREF" H 3900 2950 50  0000 C CNN
-F 2 "" H 3900 3100 50  0001 C CNN
-F 3 "" H 3900 3100 50  0001 C CNN
-	1    3900 3100
+P 4150 1500
+F 0 "#PWR6" H 4150 1250 50  0001 C CNN
+F 1 "GNDREF" H 4150 1350 50  0000 C CNN
+F 2 "" H 4150 1500 50  0001 C CNN
+F 3 "" H 4150 1500 50  0001 C CNN
+	1    4150 1500
 	1    0    0    -1
 $EndComp
@@
 L +5V #PWR7
 U 1 1 5A195FAB
-P 4400 2600
-F 0 "#PWR7" H 4400 2450 50  0001 C CNN
-F 1 "+5V" H 4400 2740 50  0000 C CNN
-F 2 "" H 4400 2600 50  0001 C CNN
-F 3 "" H 4400 2600 50  0001 C CNN
-	1    4400 2600
+P 4650 1000
+F 0 "#PWR7" H 4650 850 50  0001 C CNN
+F 1 "+5V" H 4650 1140 50  0000 C CNN
+F 2 "" H 4650 1000 50  0001 C CNN
+F 3 "" H 4650 1000 50  0001 C CNN
+	1    4650 1000
 	1    0    0    -1
 $EndComp
 Wire Wire Line
-	4200 2600 4400 2600
+	4450 1000 4650 1000
 Wire Wire Line
-	3600 2600 3400 2600
+	3850 1000 3650 1000
 Wire Wire Line
-	3900 3000 3900 3100
+	4150 1400 4150 1500
+Wire Wire Line
+	4150 1450 4550 1450
+Wire Wire Line
+	4550 1450 4550 1100
+Wire Wire Line
+	4550 1100 4450 1100
+Connection ~ 4150 1450
 $EndSCHEMATC
